File: schematic/rtty-transmitter.kicad_pcb (KiCad board)
At the start: 2 copper layers, 120 x 60 mm, 75 parts, among them J1 USB Type B Connector, J2 USBasp header, J3 2x5 Pin Header Connector Fema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, J4 Conn_01x02_Pin, J5 Conn_01x02_Pin, J6 Conn_01x02_Pin, J7 SMA Vertical Female, Q1 PN2222A, Q2 PN2222A, U1 MCP2221AxP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

Commit message: White status LED current limiting resistor changed from 470R to 1k
Parts:
- R6: value 470R -> 1k; footprint StockLib:R_470_Axial_DIN0207 -> StockLib:R_1k_Axial_DIN0207
Changed lines of the file:
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@@
 		)
 	)
-	(footprint "StockLib:R_470_Axial_DIN0207"
+	(footprint "StockLib:R_1k_Axial_DIN0207"
 		(layer "F.Cu")
 		(at 43.434 55.88)
@@
 			)
 		)
-		(property "Value" "470R"
+		(property "Value" "1k"
 			(at 5.08 2.37 0)
 			(layer "F.Fab")
@@
 		)
 		(embedded_fonts no)
-		(model "C:/Users/bazsi/Documents/KiCad/7.0/3dmodels/Resistors/Res-10.16-6.3x2.3-470.step"
+		(model "${KICAD_USER_3DMODEL_DIR}/Resistors/Res-10.16-6.3x2.3-1k.step"
 			(offset
 				(xyz 5 0 0)
